Commit message: moveit gazebo sim test 3

File: multiarm_H1/h1_description/urdf/h1.urdf (robot description, URDF)
Before this commit: robot h1_robot, 22 links, 21 joints
Links:
- added link R_hand_base_link, mass 0.14143; collision mesh filename=file:///home/robotck/ros2_ws/install/inspire_hand_descripti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; visual mesh filename=file:///home/robotck/ros2_ws/install/inspire_hand_descripti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
- added link R_index_intermediate, mass 0.0045683; collision mesh filename=file:///home/robotck/ros2_ws/install/inspire_hand_descripti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; visual mesh filename=file:///home/robotck/ros2_ws/install/inspire_hand_descripti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
- added link R_index_proximal, mass 0.0042403; collision mesh filename=file:///home/robotck/ros2_ws/install/inspire_hand_descripti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; visual mesh filename=file:///home/robotck/ros2_ws/install/inspire_hand_descripti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
- added link R_middle_intermediate, mass 0.0050396; collision mesh filename=file:///home/robotck/ros2_ws/install/inspire_hand_descripti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; visual mesh filename=file:///home/robotck/ros2_ws/install/inspire_hand_descripti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
- added link R_middle_proximal, mass 0.0042403; collision mesh filename=file:///home/robotck/ros2_ws/install/inspire_hand_descripti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; visual mesh filename=file:///home/robotck/ros2_ws/install/inspire_hand_descripti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
- added link R_pinky_intermediate, mass 0.0035996; collision mesh filename=file:///home/robotck/ros2_ws/install/inspire_hand_descripti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; visual mesh filename=file:///home/robotck/ros2_ws/install/inspire_hand_descripti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
- added link R_pinky_proximal, mass 0.0042403; collision mesh filename=file:///home/robotck/ros2_ws/install/inspire_hand_descripti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; visual mesh filename=file:///home/robotck/ros2_ws/install/inspire_hand_descripti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
- added link R_ring_intermediate, mass 0.0045683; collision mesh filename=file:///home/robotck/ros2_ws/install/inspire_hand_descripti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; visual mesh filename=file:///home/robotck/ros2_ws/install/inspire_hand_descripti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
- added link R_ring_proximal, mass 0.0042403; collision mesh filename=file:///home/robotck/ros2_ws/install/inspire_hand_descripti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; visual mesh filename=file:///home/robotck/ros2_ws/install/inspire_hand_descripti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
- added link R_thumb_distal, mass 0.0033441; collision mesh filename=file:///home/robotck/ros2_ws/install/inspire_hand_descripti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; visual mesh filename=file:///home/robotck/ros2_ws/install/inspire_hand_descripti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
- added link R_thumb_intermediate, mass 0.0037847; collision mesh filename=file:///home/robotck/ros2_ws/install/inspire_hand_descripti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; visual mesh filename=file:///home/robotck/ros2_ws/install/inspire_hand_descripti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
- added link R_thumb_proximal, mass 0.0066075; collision mesh filename=file:///home/robotck/ros2_ws/install/inspire_hand_descripti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; visual mesh filename=file:///home/robotck/ros2_ws/install/inspire_hand_descripti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
- added link R_thumb_proximal_base, mass 0.0018869; collision mesh filename=file:///home/robotck/ros2_ws/install/inspire_hand_descripti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; visual mesh filename=file:///home/robotck/ros2_ws/install/inspire_hand_descripti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
- added link hand_e_link, mass 0.86387; collision mesh filename=file:///home/robotck/ros2_ws/install/robotiq_gripper_descri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 scale=1.0 1.0 1.0; visual mesh filename=file:///home/robotck/ros2_ws/install/robotiq_gripper_descri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 scale=1.0 1.0 1.0
- added link hande_left_finger, mass 0.03804; collision mesh filename=file:///home/robotck/ros2_ws/install/robotiq_gripper_descri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 scale=1.0 1.0 1.0; visual mesh filename=file:///home/robotck/ros2_ws/install/robotiq_gripper_descri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 scale=1.0 1.0 1.0
- added link hande_right_finger, mass 0.03804; collision mesh filename=file:///home/robotck/ros2_ws/install/robotiq_gripper_descri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 scale=1.0 1.0 1.0; visual mesh filename=file:///home/robotck/ros2_ws/install/robotiq_gripper_descri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 scale=1.0 1.0 1.0
Joints:
- added joint R_index_intermediate_joint: type revolute, parent R_index_proximal, child R_index_intermediate, origin xyz=-0.0026138 0.032026 -0.001 rpy=0 0 0, axis 0 0 1, limit lower=0 upper=1.7 effort=1 velocity=0.5, mimic joint=hand_joint4 multiplier=1 offset=0
- added joint R_middle_intermediate_joint: type revolute, parent R_middle_proximal, child R_middle_intermediate, origin xyz=-0.0024229 0.032041 -0.001 rpy=0 0 0, axis 0 0 1, limit lower=0 upper=1.7 effort=1 velocity=0.5, mimic joint=hand_joint3 multiplier=1 offset=0
- added joint R_pinky_intermediate_joint: type revolute, parent R_pinky_proximal, child R_pinky_intermediate, origin xyz=-0.0024229 0.032041 -0.001 rpy=0 0 0, axis 0 0 1, limit lower=0 upper=1.7 effort=1 velocity=0.5, mimic joint=hand_joint1 multiplier=1 offset=0
- added joint R_ring_intermediate_joint: type revolute, parent R_ring_proximal, child R_ring_intermediate, origin xyz=-0.0024229 0.032041 -0.001 rpy=0 0 0, axis 0 0 1, limit lower=0 upper=1.7 effort=1 velocity=0.5, mimic joint=hand_joint2 multiplier=1 offset=0
- added joint R_thumb_distal_joint: type revolute, parent R_thumb_intermediate, child R_thumb_distal, origin xyz=0.020248 0.010156 -0.0012 rpy=0 0 0, axis 0 0 1, limit lower=0 upper=1.2 effort=1 velocity=0.5, mimic joint=hand_joint5 multiplier=2.4 offset=0
- added joint R_thumb_intermediate_joint: type revolute, parent R_thumb_proximal, child R_thumb_intermediate, origin xyz=0.04407 0.034553 -0.0008 rpy=0 0 0, axis 0 0 1, limit lower=0 upper=0.8 effort=1 velocity=0.5, mimic joint=hand_joint5 multiplier=1.6 offset=0
- added joint gripper_connect_joint: type fixed, parent link-L7, child hand_e_link, origin xyz=0 0 0 rpy=0 0 0
- added joint gripper_joint: type prismatic, parent hand_e_link, child hande_left_finger, origin xyz=0 0 0.099 rpy=0 0 0, axis -1 0 0, limit lower=0 upper=0.025 effort=130 velocity=0.15
- added joint hand_connect_joint: type fixed, parent link-R7, child R_hand_base_link, origin xyz=0 0 0 rpy=-1.57 0 1.57
- added joint hand_joint1: type revolute, parent R_hand_base_link, child R_pinky_proximal, origin xyz=0.00028533 -0.13571 0.025488 rpy=3.0369 0 0, axis 0 0 1, limit lower=0 upper=1.7 effort=1 velocity=0.5
- added joint hand_joint2: type revolute, parent R_hand_base_link, child R_ring_proximal, origin xyz=0.00028533 -0.13691 0.0062872 rpy=3.0892 0 0, axis 0 0 1, limit lower=0 upper=1.7 effort=1 velocity=0.5
- added joint hand_joint3: type revolute, parent R_hand_base_link, child R_middle_proximal, origin xyz=0.00028533 -0.1371 -0.01295 rpy=-3.1416 0 0, axis 0 0 1, limit lower=0 upper=1.7 effort=1 velocity=0.5
- added joint hand_joint4: type revolute, parent R_hand_base_link, child R_index_proximal, origin xyz=0.00028533 -0.13653 -0.032268 rpy=-3.1067 0 0, axis 0 0 1, limit lower=0 upper=1.7 effort=1 velocity=0.5
- added joint hand_joint5: type revolute, parent R_thumb_proximal_base, child R_thumb_proximal, origin xyz=-0.0088099 0.010892 -0.00925 rpy=1.5708 0 2.8587, axis 0 0 1, limit lower=-0.1 upper=0.6 effort=1 velocity=0.5
- added joint hand_joint6: type revolute, parent R_hand_base_link, child R_thumb_proximal_base, origin xyz=-0.01696 -0.0691 -0.02045 rpy=1.5708 -1.5708 0, axis 0 0 -1, limit lower=-0.1 upper=1.3 effort=1 velocity=0.5
- added joint hande_right_finger_joint: type prismatic, parent hand_e_link, child hande_right_finger, origin xyz=0 0 0.099 rpy=0 0 0, axis 1 0 0, limit lower=0 upper=0.025 effort=130 velocity=0.15, mimic joint=gripper_joint multiplier=1 offset=0
- joint Body: origin xyz=0 0 0 rpy=1.5708 0 0 -> xyz=0 0  0 rpy=1.5708 0 0
- joint J1: origin xyz=0 0 0 rpy=0 0 0 -> xyz=0 0 0.2605 rpy=0 0 0

File: multiarm_H1/h1_description/urdf/h1_ros2_control.xacro (robot description, xacro)
@@ -87,4 +87,5 @@
         <xacro:macro name ="external_device_joint_interface" params="Joint_Name initial_pos ">
           <joint name="${Joint_Name}">
+              <command_interface name="position"/>
               <state_interface name="position">
                   <param name="initial_value">${initial_pos}</param>
