Commit message: add collision detect module

File: multiarm_H1/h1_description/urdf/h1.urdf.xacro (robot description, xacro)
@@ -1213,3 +1213,21 @@
       velocity="0" />
   </joint>
+  <xacro:macro name="h1_robot_urdf_config" params="if_add_external_device">
+    <xacro:if value="${if_add_external_device}">
+      <xacro:include filename="$(find inspire_hand_description)/urdf/inspire_hand.urdf.xacro"/>
+      <xacro:include filename="$(find robotiq_gripper_description)/urdf/robotiq_gripper.urdf.xacro"/>
+      <joint name="gripper_connect_joint" type="fixed">
+        <origin xyz="0 0 0" rpy="0 0 0" />
+        <!-- <origin xyz="0 0 0.00695" rpy="0 0 0" /> -->
+        <parent link="link-L7"/>
+        <child link="hand_e_link"/>
+      </joint>
+      <joint name="hand_connect_joint" type="fixed">
+        <!-- <origin xyz="0 0 0" rpy="-1.57 0 -1.57" /> -->
+        <origin xyz="0 0 0" rpy="-1.57 0 1.57" />
+        <parent link="link-R7"/>
+        <child link="R_hand_base_link"/>
+      </joint>
+    </xacro:if>
+  </xacro:macro>
 </robot>

File: multiarm_H1/h1_description/urdf/h1.xacro (robot description, xacro)
@@ -1,5 +1,4 @@
 <?xml version="1.0" encoding="UTF-8"?>
 <robot name="h1_robot" xmlns:xacro="http://wiki.ros.org/xacro" >
-  <xacro:include filename="$(find h1_description)/urdf/h1.urdf.xacro"/>
   <xacro:arg name="sim_gazebo_classic" default="false" />
   <xacro:arg name="device_mode" default="8" />
@@ -7,6 +6,10 @@
   <xacro:arg name="system_arg" default="--path /home/robot/Work/system/robot_config --iscopy true" />
   <xacro:arg name="if_add_axisgroups" default="true" />
-  <xacro:arg name="if_add_external_device" default="true" />
+  <xacro:arg name="if_add_external_device" default="false" />
   <xacro:arg name="external_device_dof" default="7" />
+  <xacro:include filename="$(find h1_description)/urdf/h1.urdf.xacro"/>
+  <xacro:h1_robot_urdf_config
+    if_add_external_device="$(arg if_add_external_device)"
+  />
   <xacro:include filename="$(find h1_description)/urdf/h1_ros2_control.xacro"/>
   <xacro:h1_robot_ros2_control_config

File: multiarm_H1/h1_description/urdf/h1_ros2_control.xacro (robot description, xacro)
@@ -51,18 +51,20 @@
       <xacro:joint_interface Joint_Name="H-J1" initial_pos="0.0" initial_vel="0.0" initial_effort="0.0"/>
       <xacro:joint_interface Joint_Name="H-J2" initial_pos="0.0" initial_vel="0.0" initial_effort="0.0"/>
-      <xacro:macro name ="external_device_joint_interface" params="Joint_Name initial_pos ">
-        <joint name="${Joint_Name}">
-            <state_interface name="position">
-                <param name="initial_value">${initial_pos}</param>
-            </state_interface>
-        </joint>
-      </xacro:macro>
-      <xacro:external_device_joint_interface Joint_Name="hand_joint1" initial_pos="0.0" />
-      <xacro:external_device_joint_interface Joint_Name="hand_joint2" initial_pos="0.0" />
-      <xacro:external_device_joint_interface Joint_Name="hand_joint3" initial_pos="0.0" />
-      <xacro:external_device_joint_interface Joint_Name="hand_joint4" initial_pos="0.0" />
-      <xacro:external_device_joint_interface Joint_Name="hand_joint5" initial_pos="0.0" />
-      <xacro:external_device_joint_interface Joint_Name="hand_joint6" initial_pos="0.0" />
-      <xacro:external_device_joint_interface Joint_Name="gripper_joint" initial_pos="0.0" />
+      <xacro:if value="${if_add_external_device}">
+        <xacro:macro name ="external_device_joint_interface" params="Joint_Name initial_pos ">
+          <joint name="${Joint_Name}">
+              <state_interface name="position">
+                  <param name="initial_value">${initial_pos}</param>
+              </state_interface>
+          </joint>
+        </xacro:macro>
+        <xacro:external_device_joint_interface Joint_Name="hand_joint1" initial_pos="0.0" />
+        <xacro:external_device_joint_interface Joint_Name="hand_joint2" initial_pos="0.0" />
+        <xacro:external_device_joint_interface Joint_Name="hand_joint3" initial_pos="0.0" />
+        <xacro:external_device_joint_interface Joint_Name="hand_joint4" initial_pos="0.0" />
+        <xacro:external_device_joint_interface Joint_Name="hand_joint5" initial_pos="0.0" />
+        <xacro:external_device_joint_interface Joint_Name="hand_joint6" initial_pos="0.0" />
+        <xacro:external_device_joint_interface Joint_Name="gripper_joint" initial_pos="0.0" />
+      </xacro:if>
     </ros2_control>
   </xacro:macro>

Commit message: moveit gazebo sim test 1

File: multiarm_H1/h1_description/urdf/h1.urdf.xacro (robot description, xacro)
@@ -35,6 +35,9 @@
     </inertial>
     <visual>
-      <origin
-        xyz="0 0 0"
+      <!-- <origin
+        xyz="0 0 0"
+        rpy="0 0 0" /> -->
+      <origin
+        xyz="0 0 0.2605"
         rpy="0 0 0" />
       <geometry>
@@ -49,6 +52,9 @@
     </visual>
     <collision>
-      <origin
-        xyz="0 0 0"
+      <!-- <origin
+        xyz="0 0 0"
+        rpy="0 0 0" /> -->
+      <origin
+        xyz="0 0 0.2605"
         rpy="0 0 0" />
       <geometry>
@@ -101,6 +107,9 @@
     name="J1"
     type="revolute">
-    <origin
+    <!-- <origin
       xyz="0 0 0"
+      rpy="0 0 0" /> -->
+    <origin
+      xyz="0 0 0.2605"
       rpy="0 0 0" />
     <parent
@@ -160,5 +169,5 @@
     type="revolute">
     <origin
-      xyz="0 0 0"
+      xyz="0 0  0"
       rpy="1.5708 0 0" />
     <parent
@@ -1231,3 +1240,12 @@
     </xacro:if>
   </xacro:macro>
+  <xacro:macro name="gazebo_urdf_config" params="sim_gazebo_classic">
+    <xacro:if value="${sim_gazebo_classic}">
+      <link name="world"/>
+      <joint name="fixed" type="fixed">
+        <parent link="world"/>
+        <child link="fake_link"/>
+      </joint>
+    </xacro:if>
+  </xacro:macro>
 </robot>

File: multiarm_H1/h1_description/urdf/h1.xacro (robot description, xacro)
@@ -1,5 +1,5 @@
 <?xml version="1.0" encoding="UTF-8"?>
 <robot name="h1_robot" xmlns:xacro="http://wiki.ros.org/xacro" >
-  <xacro:arg name="sim_gazebo_classic" default="false" />
+  <xacro:arg name="sim_gazebo_classic" default="true" />
   <xacro:arg name="device_mode" default="8" />
   <xacro:arg name="sim_flag" default="false" />
@@ -9,7 +9,6 @@
   <xacro:arg name="external_device_dof" default="7" />
   <xacro:include filename="$(find h1_description)/urdf/h1.urdf.xacro"/>
-  <xacro:h1_robot_urdf_config
-    if_add_external_device="$(arg if_add_external_device)"
-  />
+  <xacro:h1_robot_urdf_config if_add_external_device="$(arg if_add_external_device)"/>
+  <xacro:gazebo_urdf_config sim_gazebo_classic="$(arg sim_gazebo_classic)"/>
   <xacro:include filename="$(find h1_description)/urdf/h1_ros2_control.xacro"/>
   <xacro:h1_robot_ros2_control_config

File: multiarm_H1/h1_description/urdf/h1_ros2_control.xacro (robot description, xacro)
@@ -2,4 +2,37 @@
 <robot xmlns:xacro="http://wiki.ros.org/xacro">
   <xacro:macro name="h1_robot_ros2_control_config" params="sim_gazebo_classic device_mode sim_flag system_arg if_add_axisgroups if_add_external_device external_device_dof">
+    <xacro:if value="${sim_gazebo_classic}">
+      <gazebo>
+        <plugin name="gazebo_ros2_control" filename="libgazebo_ros2_control.so">
+          <parameters>$(find hyy_hardware_driver)/config/h1_controller.yaml</parameters>
+        </plugin>
+      </gazebo>
+      <xacro:macro name ="link_reference" params="link_name material_">
+        <gazebo reference="${link_name}">
+          <material>${material_}</material>
+        </gazebo>
+      </xacro:macro>
+      <xacro:link_reference link_name="base_link" material_= "Gazebo/DarkGrey"/>
+      <xacro:link_reference link_name="link-J1" material_= "Gazebo/Orange"/>
+      <xacro:link_reference link_name="link-Body" material_= "Gazebo/DarkGrey"/>
+      <xacro:link_reference link_name="link-L0" material_= "Gazebo/White"/>
+      <xacro:link_reference link_name="link-L1" material_= "Gazebo/Grey"/>
+      <xacro:link_reference link_name="link-L2" material_= "Gazebo/White"/>
+      <xacro:link_reference link_name="link-L3" material_= "Gazebo/Grey"/>
+      <xacro:link_reference link_name="link-L4" material_= "Gazebo/White"/>
+      <xacro:link_reference link_name="link-L5" material_= "Gazebo/Grey"/>
+      <xacro:link_reference link_name="link-L6" material_= "Gazebo/White"/>
+      <xacro:link_reference link_name="link-L7" material_= "Gazebo/Grey"/>
+      <xacro:link_reference link_name="link-R0" material_= "Gazebo/White"/>
+      <xacro:link_reference link_name="link-R1" material_= "Gazebo/Grey"/>
+      <xacro:link_reference link_name="link-R2" material_= "Gazebo/White"/>
+      <xacro:link_reference link_name="link-R3" material_= "Gazebo/Grey"/>
+      <xacro:link_reference link_name="link-R4" material_= "Gazebo/White"/>
+      <xacro:link_reference link_name="link-R5" material_= "Gazebo/Grey"/>
+      <xacro:link_reference link_name="link-R6" material_= "Gazebo/White"/>
+      <xacro:link_reference link_name="link-R7" material_= "Gazebo/Grey"/>
+      <xacro:link_reference link_name="link-H0" material_= "Gazebo/White"/>
+      <xacro:link_reference link_name="link-H1" material_= "Gazebo/Grey"/>
+    </xacro:if>
     <ros2_control name="h1_robot_ros2_control" type="system">
       <hardware>

Commit message: add moveit2 program

File: multiarm_H1/h1_description/urdf/h1.urdf.xacro (robot description, xacro)
@@ -3,5 +3,5 @@
      Commit Version: 1.5.1-0-g916b5db  Build Version: 1.5.7152.31018
      For more information, please see http://wiki.ros.org/sw_urdf_exporter -->
-<robot name="h1_robot" xmlns:xacro="http://ros.org/wiki/xacro">
+<robot name="h1" xmlns:xacro="http://ros.org/wiki/xacro">
   <xacro:property name = "pkg_address" value = "file://$(find h1_description)"/>
   <link name="fake_link">
@@ -1222,30 +1222,3 @@
       velocity="0" />
   </joint>
-  <xacro:macro name="h1_robot_urdf_config" params="if_add_external_device">
-    <xacro:if value="${if_add_external_device}">
-      <xacro:include filename="$(find inspire_hand_description)/urdf/inspire_hand.urdf.xacro"/>
-      <xacro:include filename="$(find robotiq_gripper_description)/urdf/robotiq_gripper.urdf.xacro"/>
-      <joint name="gripper_connect_joint" type="fixed">
-        <origin xyz="0 0 0" rpy="0 0 0" />
-        <!-- <origin xyz="0 0 0.00695" rpy="0 0 0" /> -->
-        <parent link="link-L7"/>
-        <child link="hand_e_link"/>
-      </joint>
-      <joint name="hand_connect_joint" type="fixed">
-        <!-- <origin xyz="0 0 0" rpy="-1.57 0 -1.57" /> -->
-        <origin xyz="0 0 0" rpy="-1.57 0 1.57" />
-        <parent link="link-R7"/>
-        <child link="R_hand_base_link"/>
-      </joint>
-    </xacro:if>
-  </xacro:macro>
-  <xacro:macro name="gazebo_urdf_config" params="sim_gazebo_classic">
-    <xacro:if value="${sim_gazebo_classic}">
-      <link name="world"/>
-      <joint name="fixed" type="fixed">
-        <parent link="world"/>
-        <child link="fake_link"/>
-      </joint>
-    </xacro:if>
-  </xacro:macro>
 </robot>

File: multiarm_H1/h1_description/urdf/h1.xacro (robot description, xacro)
@@ -6,9 +6,11 @@
   <xacro:arg name="system_arg" default="--path /home/robot/Work/system/robot_config --iscopy true" />
   <xacro:arg name="if_add_axisgroups" default="true" />
-  <xacro:arg name="if_add_external_device" default="false" />
+  <xacro:arg name="if_add_external_device" default="true" />
   <xacro:arg name="external_device_dof" default="7" />
   <xacro:include filename="$(find h1_description)/urdf/h1.urdf.xacro"/>
-  <xacro:h1_robot_urdf_config if_add_external_device="$(arg if_add_external_device)"/>
-  <xacro:gazebo_urdf_config sim_gazebo_classic="$(arg sim_gazebo_classic)"/>
+  <xacro:include filename="$(find h1_description)/urdf/gazebo_config.xacro"/>
+  <xacro:include filename="$(find h1_description)/urdf/external_devices_config.xacro"/>
+  <xacro:external_device_config if_add_external_device="$(arg if_add_external_device)"/>
+  <xacro:gazebo_config sim_gazebo_classic="$(arg sim_gazebo_classic)"/>
   <xacro:include filename="$(find h1_description)/urdf/h1_ros2_control.xacro"/>
   <xacro:h1_robot_ros2_control_config

File: multiarm_H1/h1_description/urdf/h1_robot.urdf.xacro (robot description, xacro)
@@ -1,17 +1,7 @@
 <?xml version="1.0" encoding="UTF-8"?>
-<robot name="t1_robot" xmlns:xacro="http://wiki.ros.org/xacro" >
-  <xacro:include filename="$(find h1_description)/urdf/h1.urdf.xacro"/>
-  <xacro:include filename="$(find inspire_hand_description)/urdf/inspire_hand.urdf.xacro"/>
-  <xacro:include filename="$(find robotiq_gripper_description)/urdf/robotiq_gripper.urdf.xacro"/>
-  <joint name="gripper_connect_joint" type="fixed">
-    <origin xyz="0 0 0" rpy="0 0 0" />
-    <!-- <origin xyz="0 0 0.00695" rpy="0 0 0" /> -->
-    <parent link="link-L7"/>
-    <child link="hand_e_link"/>
-  </joint>
-  <joint name="hand_connect_joint" type="fixed">
-    <origin xyz="0 0 0" rpy="-1.57 0 -1.57" />
-    <parent link="link-R7"/>
-    <child link="R_hand_base_link"/>
-  </joint>
+<robot name="h1_robot" xmlns:xacro="http://wiki.ros.org/xacro" >
+    <xacro:arg name="if_add_external_device" default="true" />
+    <xacro:include filename="$(find h1_description)/urdf/h1.urdf.xacro"/>
+    <xacro:include filename="$(find h1_description)/urdf/external_devices_config.xacro"/>
+    <xacro:external_device_config if_add_external_device="$(arg if_add_external_device)"/>
 </robot>
