Commit message: update t1 description

File: humanoid_robot/multi_arm_description/urdf/t1_robot.urdf.xacro (robot description, xacro)
@@ -1,16 +1,7 @@
 <?xml version="1.0" encoding="UTF-8"?>
 <robot name="t1_robot" xmlns:xacro="http://wiki.ros.org/xacro" >
-  <xacro:include filename="$(find multi_arm_description)/urdf/dual_arm_robot.urdf.xacro"/>
-  <xacro:include filename="$(find inspire_hand_description)/urdf/inspire_hand.urdf.xacro"/>
-  <xacro:include filename="$(find robotiq_gripper_description)/urdf/robotiq_gripper.urdf.xacro"/>
-  <joint name="gripper_connect_joint" type="fixed">
-    <origin xyz="0 0 0.00695" rpy="0 0 0" />
-    <parent link="link-Ltool"/>
-    <child link="hand_e_link"/>
-  </joint>
-  <joint name="hand_connect_joint" type="fixed">
-    <origin xyz="0 0 0" rpy="-1.57 0 -1.57" />
-    <parent link="link-Rtool"/>
-    <child link="R_hand_base_link"/>
-  </joint>
+    <xacro:arg name="if_add_external_device" default="true" />
+    <xacro:include filename="$(find multi_arm_description)/urdf/t1.urdf.xacro"/>
+    <xacro:include filename="$(find multi_arm_description)/urdf/external_devices_config.xacro"/>
+    <xacro:external_device_config if_add_external_device="$(arg if_add_external_device)"/>
 </robot>
