Commit message: add stop interface(test)

File: humanoid_robot/multi_arm_description/urdf/t1.urdf.xacro (robot description, xacro)
@@ -22,15 +22,15 @@
     <inertial>
       <origin
-        xyz="0.00608770814142283 0.00345294437108543 0.36719318766884"
-        rpy="0 0 0" />
-      <mass
-        value="5.08372108708452" />
-      <inertia
-        ixx="0.0681483796497588"
+        xyz="-0.0141157259588467 -0.016243923969749 0.343988437034855"
+        rpy="0 0 0" />
+      <mass
+        value="6.29377720970293" />
+      <inertia
+        ixx="0.0915834842999805"
         ixy="-6.583736565642E-05"
-        ixz="-0.00435126206558179"
-        iyy="0.0562781365647336"
+        ixz="-0.00435126206558178"
+        iyy="0.0797132412149553"
         iyz="-0.000288236319946359"
-        izz="0.0317831828027757" />
+        izz="0.0318440700579395" />
     </inertial>
     <visual>
@@ -62,5 +62,5 @@
     <inertial>
       <origin
-        xyz="-0.000158222660641598 -9.98278990236623E-06 -0.249624469139269"
+        xyz="-0.000158222660641603 -9.98278990237011E-06 -0.249624469139269"
         rpy="0 0 0" />
       <mass
@@ -68,8 +68,8 @@
       <inertia
         ixx="0.0248203808488518"
-        ixy="-2.36063985454879E-08"
+        ixy="-2.36063985452956E-08"
         ixz="-0.000749290486872422"
         iyy="0.01388988449036"
-        iyz="7.57304943520522E-07"
+        iyz="7.5730494352056E-07"
         izz="0.0185938049482952" />
     </inertial>
@@ -111,5 +111,5 @@
       xyz="0 0 1" />
     <limit
-      lower="0.00"
+      lower="-0.05"
       upper="0.21"
       effort="0"
@@ -120,15 +120,15 @@
     <inertial>
       <origin
-        xyz="-1.6666483421104E-05 -0.000428575028514344 0.0387665520212092"
+        xyz="0.000428575028514344 -1.66664834211078E-05 0.0387665520212092"
         rpy="0 0 0" />
       <mass
         value="4.48243687136842" />
       <inertia
-        ixx="0.00516757527508353"
-        ixy="-6.99003877944147E-07"
-        ixz="-1.89822417332752E-06"
-        iyy="0.00522193992152092"
-        iyz="-4.82183712983688E-05"
-        izz="0.00566118382384461" />
+        ixx="0.00522193992152092"
+        ixy="6.99003877943978E-07"
+        ixz="4.82183712983686E-05"
+        iyy="0.00516757527508353"
+        iyz="-1.89822417332785E-06"
+        izz="0.00566118382384462" />
     </inertial>
     <visual>
@@ -161,5 +161,5 @@
     <origin
       xyz="0 -0.09 -0.075"
-      rpy="1.5708 0 0" />
+      rpy="1.5708 1.5708 0" />
     <parent
       link="Link-Body" />
@@ -179,5 +179,5 @@
       <inertia
         ixx="0.00538935884644845"
-        ixy="-3.40948002179596E-09"
+        ixy="-3.40948002179718E-09"
         ixz="-4.54525514109768E-07"
         iyy="0.00597533433884467"
@@ -214,5 +214,5 @@
     <origin
       xyz="0 0 0.172"
-      rpy="0 0 -1.5708" />
+      rpy="0 0 0" />
     <parent
       link="link-R0" />
@@ -231,5 +231,5 @@
     <inertial>
       <origin
-        xyz="-1.21016987286726E-06 -0.0553985267336023 -0.00166564475227283"
+        xyz="-1.21016987286726E-06 -0.0553985267336023 -0.00166564475227282"
         rpy="0 0 0" />
       <mass
@@ -237,8 +237,8 @@
       <inertia
         ixx="0.0152384536230366"
-        ixy="-1.14870185368696E-06"
-        ixz="-2.6851571084856E-08"
+        ixy="-1.14870185368694E-06"
+        ixz="-2.68515710848592E-08"
         iyy="0.00674678421570552"
-        iyz="0.000400962979098618"
+        iyz="0.000400962979098617"
         izz="0.0142810956251759" />
     </inertial>
@@ -289,10 +289,10 @@
     <inertial>
       <origin
-        xyz="-0.00236928911888323 0.000256017152003125 -0.0989215512578252"
+        xyz="-0.00236928911888323 0.000256017152003125 -0.0989215512578251"
         rpy="0 0 0" />
       <mass
         value="6.76099941307626" />
       <inertia
-        ixx="0.0241007935216868"
+        ixx="0.0241007935216869"
         ixy="-4.07055219750389E-06"
         ixz="0.00052429441504994"
@@ -347,5 +347,5 @@
     <inertial>
       <origin
-        xyz="1.55020330738775E-06 -0.0327095870323233 -0.000281996819201039"
+        xyz="1.55020330738775E-06 -0.0327095870323233 -0.000281996819201036"
         rpy="0 0 0" />
       <mass
@@ -353,6 +353,6 @@
       <inertia
         ixx="0.0198391962830934"
-        ixy="-2.77202330132127E-07"
-        ixz="-1.52336964149364E-08"
+        ixy="-2.77202330132049E-07"
+        ixz="-1.52336964151243E-08"
         iyy="0.00950734139914809"
         iyz="5.51814068233546E-05"
@@ -405,12 +405,12 @@
     <inertial>
       <origin
-        xyz="2.61938777335047E-06 0.000664248517209837 -0.0552339020133823"
+        xyz="2.61938777335047E-06 0.000664248517209838 -0.0552339020133823"
         rpy="0 0 0" />
       <mass
         value="3.13715935450461" />
       <inertia
-        ixx="0.00617168729257163"
+        ixx="0.00617168729257164"
         ixy="9.57723919184407E-08"
-        ixz="-4.53982816082471E-07"
+        ixz="-4.53982816082469E-07"
         iyy="0.00650310856970505"
         iyz="-0.000114073990108045"
@@ -463,5 +463,5 @@
     <inertial>
       <origin
-        xyz="1.46922276367256E-06 -0.0320401134442209 -0.000354045768412676"
+        xyz="1.46922276367256E-06 -0.0320401134442208 -0.000354045768412677"
         rpy="0 0 0" />
       <mass
@@ -469,8 +469,8 @@
       <inertia
         ixx="0.0130568238032191"
-        ixy="-2.44895572730431E-07"
-        ixz="1.52953724925497E-07"
+        ixy="-2.44895572730433E-07"
+        ixz="1.52953724925499E-07"
         iyy="0.00624175373758098"
-        iyz="5.44179711474993E-05"
+        iyz="5.44179711474995E-05"
         izz="0.0110970473747011" />
     </inertial>
@@ -521,5 +521,5 @@
     <inertial>
       <origin
-        xyz="0.000201227208657229 -4.45951571791945E-06 -0.0324015634635619"
+        xyz="0.000201227208657229 -4.45951571791942E-06 -0.0324015634635619"
         rpy="0 0 0" />
       <mass
@@ -527,8 +527,8 @@
       <inertia
         ixx="0.00140827770383968"
-        ixy="-4.53525874180243E-09"
+        ixy="-4.53525874180464E-09"
         ixz="-1.01773030744789E-05"
         iyy="0.00142257226784241"
-        iyz="-2.4533932555503E-07"
+        iyz="-2.45339325555032E-07"
         izz="0.00166147868684454" />
     </inertial>
@@ -579,5 +579,5 @@
     <inertial>
       <origin
-        xyz="0.000108228106315056 -1.58700641768567E-05 -0.033217114965277"
+        xyz="0.000108228106315056 -1.58700646321033E-05 -0.0332171149652771"
         rpy="0 0 0" />
       <mass
@@ -585,8 +585,8 @@
       <inertia
         ixx="0.000108307997361677"
-        ixy="5.76555958161368E-08"
-        ixz="-9.61151743846956E-08"
-        iyy="0.000110720195394877"
-        iyz="-8.59971960181788E-09"
+        ixy="5.76555958161387E-08"
+        ixz="-9.61151743846959E-08"
+        iyy="0.000110720195394878"
+        iyz="-8.59971960181812E-09"
         izz="0.000197661960567637" />
     </inertial>
@@ -632,14 +632,14 @@
     <inertial>
       <origin
-        xyz="1.6666483512664E-05 0.000428575028515121 0.0387665520212093"
+        xyz="0.000428575028515121 -1.66664835126598E-05 0.0387665520212093"
         rpy="0 0 0" />
       <mass
         value="4.48243687136841" />
       <inertia
-        ixx="0.00516757527508331"
-        ixy="-6.99003877942928E-07"
-        ixz="1.89822417332268E-06"
-        iyy="0.00522193992152107"
-        iyz="4.8218371298447E-05"
+        ixx="0.00522193992152107"
+        ixy="6.99003877942915E-07"
+        ixz="4.82183712984472E-05"
+        iyy="0.00516757527508331"
+        iyz="-1.89822417332259E-06"
         izz="0.00566118382384421" />
     </inertial>
@@ -673,5 +673,5 @@
     <origin
       xyz="0 0.09 -0.075"
-      rpy="-1.5708 0 0" />
+      rpy="-1.5708 1.5708 0" />
     <parent
       link="Link-Body" />
@@ -685,5 +685,5 @@
     <inertial>
       <origin
-        xyz="3.21247853196649E-06 -0.000524470579303317 -0.0441242557403994"
+        xyz="3.21247853196649E-06 -0.000524470579303316 -0.0441242557403994"
         rpy="0 0 0" />
       <mass
@@ -691,6 +691,6 @@
       <inertia
         ixx="0.00538963812553377"
-        ixy="-3.4095024805657E-09"
-        ixz="4.5452558593587E-07"
+        ixy="-3.40950248056596E-09"
+        ixz="4.54525585935868E-07"
         iyy="0.00597561361790467"
         iyz="7.6416224176846E-05"
@@ -726,5 +726,5 @@
     <origin
       xyz="0 0 0.172"
-      rpy="0 0 1.5708" />
+      rpy="0 0 0" />
     <parent
       link="link-L0" />
@@ -743,14 +743,14 @@
     <inertial>
       <origin
-        xyz="1.21053463830734E-06 -0.0553985275990222 0.00166564644389522"
-        rpy="0 0 0" />
-      <mass
-        value="5.63523249981779" />
+        xyz="1.21053463841836E-06 -0.0553985275990222 0.00166564644389522"
+        rpy="0 0 0" />
+      <mass
+        value="5.63523249981778" />
       <inertia
         ixx="0.0152384532072431"
-        ixy="1.14857930990107E-06"
-        ixz="-2.69260236187485E-08"
+        ixy="1.14857930990098E-06"
+        ixz="-2.6926023618803E-08"
         iyy="0.00674678405526804"
-        iyz="-0.000400962800547985"
+        iyz="-0.000400962800547983"
         izz="0.0142810952659943" />
     </inertial>
@@ -862,10 +862,10 @@
         rpy="0 0 0" />
       <mass
-        value="6.86474389336079" />
+        value="6.8647438933608" />
       <inertia
         ixx="0.0198391959633156"
-        ixy="2.7718149887142E-07"
-        ixz="-1.54048707117146E-08"
-        iyy="0.00950734101323493"
+        ixy="2.77181498871418E-07"
+        ixz="-1.54048707117185E-08"
+        iyy="0.00950734101323492"
         iyz="-5.51813656186912E-05"
         izz="0.0163570914575466" />
@@ -923,9 +923,9 @@
       <inertia
         ixx="0.00617168729256577"
-        ixy="9.57723801003195E-08"
-        ixz="4.53982841712059E-07"
+        ixy="9.57723801003196E-08"
+        ixz="4.53982841712062E-07"
         iyy="0.00650310856968162"
-        iyz="0.000114073990132104"
-        izz="0.0020759923502868" />
+        iyz="0.000114073990132103"
+        izz="0.00207599235028679" />
     </inertial>
     <visual>
@@ -975,5 +975,5 @@
     <inertial>
       <origin
-        xyz="-1.46922276367256E-06 -0.0320401134442212 0.000354045767970296"
+        xyz="-1.46922276367256E-06 -0.0320401134442211 0.000354045767970301"
         rpy="0 0 0" />
       <mass
@@ -981,8 +981,8 @@
       <inertia
         ixx="0.0130568238032191"
-        ixy="2.4489557274105E-07"
-        ixz="1.5295372493794E-07"
+        ixy="2.44895572741051E-07"
+        ixz="1.52953724937942E-07"
         iyy="0.00624175373758096"
-        iyz="-5.44179711474942E-05"
+        iyz="-5.44179711474945E-05"
         izz="0.0110970473747011" />
     </inertial>
@@ -1033,5 +1033,5 @@
     <inertial>
       <origin
-        xyz="0.000201227208658783 -4.45951226892605E-06 -0.0324015634635619"
+        xyz="0.000201227208658783 -4.45951226892607E-06 -0.0324015634635619"
         rpy="0 0 0" />
       <mass
@@ -1039,8 +1039,8 @@
       <inertia
         ixx="0.00140827770383969"
-        ixy="-4.53525875977876E-09"
+        ixy="-4.53525875977644E-09"
         ixz="-1.01773030744803E-05"
         iyy="0.00142257226784241"
-        iyz="-2.4533932510959E-07"
+        iyz="-2.45339325109591E-07"
         izz="0.00166147868684455" />
     </inertial>
@@ -1091,14 +1091,14 @@
     <inertial>
       <origin
-        xyz="0.000109753641508337 -1.6093767850178E-05 -0.0269481337256603"
+        xyz="0.000109753641508337 -1.60937678912339E-05 -0.0269481337256519"
         rpy="0 0 0" />
       <mass
         value="0.230700440407675" />
       <inertia
-        ixx="0.000104208489619373"
-        ixy="5.76643215390902E-08"
-        ixz="-6.47742951675152E-08"
+        ixx="0.000104208489619374"
+        ixy="5.76643215390994E-08"
+        ixz="-6.47742951675387E-08"
         iyy="0.000106620567904689"
-        iyz="-3.13502539431154E-09"
+        iyz="-3.13502539430455E-09"
         izz="0.000192988356501623" />
     </inertial>
@@ -1150,5 +1150,5 @@
       <inertia
         ixx="2.39224248667145E-05"
-        ixy="-1.46844515801986E-07"
+        ixy="-1.46844515801985E-07"
         ixz="-2.53729271028935E-06"
         iyy="3.68919711015593E-05"
@@ -1202,5 +1202,5 @@
     <inertial>
       <origin
-        xyz="0.0207949033546781 -0.0845619965913866 0.000741712456379605"
+        xyz="0.0207949033546969 -0.0845619965913866 0.000741712456376936"
         rpy="0 0 0" />
       <mass
@@ -1211,5 +1211,5 @@
         ixz="1.91808717006784E-06"
         iyy="0.00152247523425536"
-        iyz="8.46665148980836E-07"
+        iyz="8.46665148980628E-07"
         izz="0.000842200739248113" />
     </inertial>
@@ -1260,15 +1260,15 @@
     <inertial>
       <origin
-        xyz="0.0322543986624866 6.03314827074541E-05 -0.0125498678920444"
-        rpy="0 0 0" />
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