Commit message: add robot_ok and modify demos

File: external_device/inspire_hand_description/urdf/inspire_hand.urdf.xacro (robot description, xacro)
@@ -37,19 +37,19 @@
       <geometry>
         <mesh
-          filename="${pkg_address}/meshes/visual/base_link.STL" />
-      </geometry>
-      <material
-        name="">
-        <color
-          rgba="1 1 1 1" />
-      </material>
-    </visual>
-    <collision>
-      <origin
-        xyz="0 0 0"
-        rpy="0 0 0" />
-      <geometry>
-        <mesh
-          filename="${pkg_address}/meshes/visual/base_link.STL" />
+          filename="${pkg_address}/meshes/visual/R_hand_base_link.STL" />
+      </geometry>
+      <material
+        name="">
+        <color
+          rgba="1 1 1 1" />
+      </material>
+    </visual>
+    <collision>
+      <origin
+        xyz="0 0 0"
+        rpy="0 0 0" />
+      <geometry>
+        <mesh
+          filename="${pkg_address}/meshes/visual/R_hand_base_link.STL" />
       </geometry>
     </collision>

File: humanoid_robot/multi_arm_description/urdf/t1.urdf.xacro (robot description, xacro)
@@ -109,8 +109,8 @@
       link="Link-Body" />
     <axis
-      xyz="0 0 1" />
-    <limit
-      lower="-0.05"
-      upper="0.21"
+      xyz="0 0 -1" />
+    <limit
+      lower="-0.15"
+      upper="0.0"
       effort="0"
       velocity="0" />
@@ -222,6 +222,6 @@
       xyz="0 0 1" />
     <limit
-      lower="-3.0543"
-      upper="3.0543"
+      lower="-3.0"
+      upper="3.0"
       effort="0"
       velocity="0" />
@@ -280,6 +280,6 @@
       xyz="0 0 1" />
     <limit
-      lower="-1.8246"
-      upper="1.8246"
+      lower="-1.6"
+      upper="1.6"
       effort="0"
       velocity="0" />
@@ -338,6 +338,6 @@
       xyz="0 0 1" />
     <limit
-      lower="-3.0543"
-      upper="3.0543"
+      lower="-3.0"
+      upper="3.0"
       effort="0"
       velocity="0" />
@@ -396,6 +396,6 @@
       xyz="0 0 1" />
     <limit
-      lower="-2.3538"
-      upper="1.7123"
+      lower="-1.7"
+      upper="2.2"
       effort="0"
       velocity="0" />
@@ -454,6 +454,6 @@
       xyz="0 0 1" />
     <limit
-      lower="-3.0543"
-      upper="3.0543"
+      lower="-3.0"
+      upper="3.0"
       effort="0"
       velocity="0" />
@@ -512,6 +512,6 @@
       xyz="0 0 1" />
     <limit
-      lower="-2.0944"
-      upper="2.0944"
+      lower="-2.0"
+      upper="2.0"
       effort="0"
       velocity="0" />
@@ -570,6 +570,6 @@
       xyz="0 0 1" />
     <limit
-      lower="-3.0543"
-      upper="3.0543"
+      lower="-3.0"
+      upper="3.0"
       effort="0"
       velocity="0" />
@@ -734,6 +734,6 @@
       xyz="0 0 1" />
     <limit
-      lower="-3.0543"
-      upper="3.0543"
+      lower="-3.0"
+      upper="3.0"
       effort="0"
       velocity="0" />
@@ -792,6 +792,6 @@
       xyz="0 0 1" />
     <limit
-      lower="-1.8246"
-      upper="1.8246"
+      lower="-1.6"
+      upper="1.6"
       effort="0"
       velocity="0" />
@@ -850,6 +850,6 @@
       xyz="0 0 1" />
     <limit
-      lower="-3.0543"
-      upper="3.0543"
+      lower="-3.0"
+      upper="3.0"
       effort="0"
       velocity="0" />
@@ -908,6 +908,6 @@
       xyz="0 0 1" />
     <limit
-      lower="-2.3538"
-      upper="1.7123"
+      lower="-1.7"
+      upper="2.2"
       effort="0"
       velocity="0" />
@@ -966,6 +966,6 @@
       xyz="0 0 1" />
     <limit
-      lower="-3.0543"
-      upper="3.0543"
+      lower="-3.0"
+      upper="3.0"
       effort="0"
       velocity="0" />
@@ -1024,6 +1024,6 @@
       xyz="0 0 1" />
     <limit
-      lower="-2.0944"
-      upper="2.0944"
+      lower="-2.0"
+      upper="2.0"
       effort="0"
       velocity="0" />
@@ -1082,6 +1082,6 @@
       xyz="0 0 1" />
     <limit
-      lower="-3.0543"
-      upper="3.0543"
+      lower="-3.0"
+      upper="3.0"
       effort="0"
       velocity="0" />
@@ -1193,6 +1193,6 @@
       xyz="0 0 1" />
     <limit
-      lower="-3.14"
-      upper="3.14"
+      lower="-1.5"
+      upper="1.5"
       effort="0"
       velocity="0" />
@@ -1251,6 +1251,6 @@
       xyz="0 0 1" />
     <limit
-      lower="-1.5708"
-      upper="1.5708"
+      lower="-0.6"
+      upper="0.6"
       effort="0"
       velocity="0" />
