Commit message: complete hyy_actions moveXYZW_action

File: robot_description/h1_description/urdf/h1.urdf (robot description, URDF)
Before this commit: robot h1_robot, 22 links, 21 joints
Links:
- link base_link: geometry collision mesh filename=file:///home/robotck/ros2_ws/install/h1_description/share/h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; visual mesh filename=file:///home/robotck/ros2_ws/install/h1_description/share/h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
- link link-Body: geometry collision mesh filename=file:///home/robotck/ros2_ws/install/h1_description/share/h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; visual mesh filename=file:///home/robotck/ros2_ws/install/h1_description/share/h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
- link link-H0: geometry collision mesh filename=file:///home/robotck/ros2_ws/install/h1_description/share/h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; visual mesh filename=file:///home/robotck/ros2_ws/install/h1_description/share/h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
- link link-H1: geometry collision mesh filename=file:///home/robotck/ros2_ws/install/h1_description/share/h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; visual mesh filename=file:///home/robotck/ros2_ws/install/h1_description/share/h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
- link link-J1: geometry collision mesh filename=file:///home/robotck/ros2_ws/install/h1_description/share/h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; visual mesh filename=file:///home/robotck/ros2_ws/install/h1_description/share/h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
- link link-L0: geometry collision mesh filename=file:///home/robotck/ros2_ws/install/h1_description/share/h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; visual mesh filename=file:///home/robotck/ros2_ws/install/h1_description/share/h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
- link link-L1: geometry collision mesh filename=file:///home/robotck/ros2_ws/install/h1_description/share/h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; visual mesh filename=file:///home/robotck/ros2_ws/install/h1_description/share/h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
- link link-L2: geometry collision mesh filename=file:///home/robotck/ros2_ws/install/h1_description/share/h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; visual mesh filename=file:///home/robotck/ros2_ws/install/h1_description/share/h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
- link link-L3: geometry collision mesh filename=file:///home/robotck/ros2_ws/install/h1_description/share/h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; visual mesh filename=file:///home/robotck/ros2_ws/install/h1_description/share/h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
- link link-L4: geometry collision mesh filename=file:///home/robotck/ros2_ws/install/h1_description/share/h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; visual mesh filename=file:///home/robotck/ros2_ws/install/h1_description/share/h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
- link link-L5: geometry collision mesh filename=file:///home/robotck/ros2_ws/install/h1_description/share/h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; visual mesh filename=file:///home/robotck/ros2_ws/install/h1_description/share/h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
- link link-L6: geometry collision mesh filename=file:///home/robotck/ros2_ws/install/h1_description/share/h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; visual mesh filename=file:///home/robotck/ros2_ws/install/h1_description/share/h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
- link link-L7: geometry collision mesh filename=file:///home/robotck/ros2_ws/install/h1_description/share/h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; visual mesh filename=file:///home/robotck/ros2_ws/install/h1_description/share/h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
- link link-R0: geometry collision mesh filename=file:///home/robotck/ros2_ws/install/h1_description/share/h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; visual mesh filename=file:///home/robotck/ros2_ws/install/h1_description/share/h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
- link link-R1: geometry collision mesh filename=file:///home/robotck/ros2_ws/install/h1_description/share/h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; visual mesh filename=file:///home/robotck/ros2_ws/install/h1_description/share/h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
- link link-R2: geometry collision mesh filename=file:///home/robotck/ros2_ws/install/h1_description/share/h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; visual mesh filename=file:///home/robotck/ros2_ws/install/h1_description/share/h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
- link link-R3: geometry collision mesh filename=file:///home/robotck/ros2_ws/install/h1_description/share/h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; visual mesh filename=file:///home/robotck/ros2_ws/install/h1_description/share/h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
- link link-R4: geometry collision mesh filename=file:///home/robotck/ros2_ws/install/h1_description/share/h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; visual mesh filename=file:///home/robotck/ros2_ws/install/h1_description/share/h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
- link link-R5: geometry collision mesh filename=file:///home/robotck/ros2_ws/install/h1_description/share/h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; visual mesh filename=file:///home/robotck/ros2_ws/install/h1_description/share/h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
- link link-R6: geometry collision mesh filename=file:///home/robotck/ros2_ws/install/h1_description/share/h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; visual mesh filename=file:///home/robotck/ros2_ws/install/h1_description/share/h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
- link link-R7: geometry collision mesh filename=file:///home/robotck/ros2_ws/install/h1_description/share/h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; visual mesh filename=file:///home/robotck/ros2_ws/install/h1_description/share/h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
Joints:
- joint J1: limit lower=-3.0543 upper=3.0543 effort=0 velocity=0 -> lower=-3.0 upper=3.0 effort=0 velocity=0
- joint L-J1: limit lower=-3.0543 upper=3.0543 effort=0 velocity=0 -> lower=-3.0 upper=3.0 effort=0 velocity=0
- joint L-J3: limit lower=-3.0543 upper=3.0543 effort=0 velocity=0 -> lower=-3.0 upper=3.0 effort=0 velocity=0
- joint L-J4: limit lower=-2.2 upper=1.7 effort=0 velocity=0 -> lower=-1.7 upper=2.2 effort=0 velocity=0
- joint L-J5: limit lower=-3.0543 upper=3.0543 effort=0 velocity=0 -> lower=-3.0 upper=3.0 effort=0 velocity=0
- joint L-J7: limit lower=-3.0543 upper=3.0543 effort=0 velocity=0 -> lower=-3.0 upper=3.0 effort=0 velocity=0
- joint R-J1: limit lower=-3.0543 upper=3.0543 effort=0 velocity=0 -> lower=-3.0 upper=3.0 effort=0 velocity=0
- joint R-J3: limit lower=-3.0543 upper=3.0543 effort=0 velocity=0 -> lower=-3.0 upper=3.0 effort=0 velocity=0
- joint R-J5: limit lower=-3.0543 upper=3.0543 effort=0 velocity=0 -> lower=-3.0 upper=3.0 effort=0 velocity=0
- joint R-J7: limit lower=-3.0543 upper=3.0543 effort=0 velocity=0 -> lower=-3.0 upper=3.0 effort=0 velocity=0

File: robot_description/h1_description/urdf/h1.urdf.xacro (robot description, xacro)
@@ -120,6 +120,6 @@
       xyz="0 0 -1" />
     <limit
-      lower="-3.0543"
-      upper="3.0543"
+      lower="-3.0"
+      upper="3.0"
       effort="0"
       velocity="0" />
@@ -294,6 +294,6 @@
       xyz="0 0 1" />
     <limit
-      lower="-3.0543"
-      upper="3.0543"
+      lower="-3.0"
+      upper="3.0"
       effort="0"
       velocity="0" />
@@ -410,6 +410,6 @@
       xyz="0 0 1" />
     <limit
-      lower="-3.0543"
-      upper="3.0543"
+      lower="-3.0"
+      upper="3.0"
       effort="0"
       velocity="0" />
@@ -526,6 +526,6 @@
       xyz="0 0 1" />
     <limit
-      lower="-3.0543"
-      upper="3.0543"
+      lower="-3.0"
+      upper="3.0"
       effort="0"
       velocity="0" />
@@ -642,6 +642,6 @@
       xyz="0 0 1" />
     <limit
-      lower="-3.0543"
-      upper="3.0543"
+      lower="-3.0"
+      upper="3.0"
       effort="0"
       velocity="0" />
@@ -753,6 +753,6 @@
       xyz="0 0 1" />
     <limit
-      lower="-3.0543"
-      upper="3.0543"
+      lower="-3.0"
+      upper="3.0"
       effort="0"
       velocity="0" />
@@ -869,6 +869,6 @@
       xyz="0 0 1" />
     <limit
-      lower="-3.0543"
-      upper="3.0543"
+      lower="-3.0"
+      upper="3.0"
       effort="0"
       velocity="0" />
@@ -927,6 +927,6 @@
       xyz="0 0 1" />
     <limit
-      lower="-2.2"
-      upper="1.7"
+      lower="-1.7"
+      upper="2.2"
       effort="0"
       velocity="0" />
@@ -985,6 +985,6 @@
       xyz="0 0 1" />
     <limit
-      lower="-3.0543"
-      upper="3.0543"
+      lower="-3.0"
+      upper="3.0"
       effort="0"
       velocity="0" />
@@ -1101,6 +1101,6 @@
       xyz="0 0 1" />
     <limit
-      lower="-3.0543"
-      upper="3.0543"
+      lower="-3.0"
+      upper="3.0"
       effort="0"
       velocity="0" />

File: robot_description/h1_description/urdf/h1_robot.urdf (robot description, URDF)
Before this commit: robot h1_robot, 38 links, 37 joints
Joints:
- joint J1: limit lower=-3.0543 upper=3.0543 effort=0 velocity=0 -> lower=-3.0 upper=3.0 effort=0 velocity=0
- joint L-J1: limit lower=-3.0543 upper=3.0543 effort=0 velocity=0 -> lower=-3.0 upper=3.0 effort=0 velocity=0
- joint L-J3: limit lower=-3.0543 upper=3.0543 effort=0 velocity=0 -> lower=-3.0 upper=3.0 effort=0 velocity=0
- joint L-J4: limit lower=-2.2 upper=1.7 effort=0 velocity=0 -> lower=-1.7 upper=2.2 effort=0 velocity=0
- joint L-J5: limit lower=-3.0543 upper=3.0543 effort=0 velocity=0 -> lower=-3.0 upper=3.0 effort=0 velocity=0
- joint L-J7: limit lower=-3.0543 upper=3.0543 effort=0 velocity=0 -> lower=-3.0 upper=3.0 effort=0 velocity=0
- joint R-J1: limit lower=-3.0543 upper=3.0543 effort=0 velocity=0 -> lower=-3.0 upper=3.0 effort=0 velocity=0
- joint R-J3: limit lower=-3.0543 upper=3.0543 effort=0 velocity=0 -> lower=-3.0 upper=3.0 effort=0 velocity=0
- joint R-J5: limit lower=-3.0543 upper=3.0543 effort=0 velocity=0 -> lower=-3.0 upper=3.0 effort=0 velocity=0
- joint R-J7: limit lower=-3.0543 upper=3.0543 effort=0 velocity=0 -> lower=-3.0 upper=3.0 effort=0 velocity=0
