Commit message: test gazebo urdf

File: robot_description/inspire_hand_description/urdf/gazebo/inspire_hand_gazebo.urdf.xacro (robot description, xacro)
@@ -37,19 +37,19 @@
       <geometry>
         <mesh
-          filename="package://inspire_hand_description/meshes/visual/R_hand_base_link.STL" />
-      </geometry>
-      <material
-        name="">
-        <color
-          rgba="1 1 1 1" />
-      </material>
-    </visual>
-    <collision>
-      <origin
-        xyz="0 0 0"
-        rpy="0 0 0" />
-      <geometry>
-        <mesh
-          filename="package://inspire_hand_description/meshes/visual/R_hand_base_link.STL" />
+          filename="${pkg_address}/meshes/visual/R_hand_base_link.STL" />
+      </geometry>
+      <material
+        name="">
+        <color
+          rgba="1 1 1 1" />
+      </material>
+    </visual>
+    <collision>
+      <origin
+        xyz="0 0 0"
+        rpy="0 0 0" />
+      <geometry>
+        <mesh
+          filename="${pkg_address}/meshes/visual/R_hand_base_link.STL" />
       </geometry>
     </collision>
@@ -77,19 +77,19 @@
       <geometry>
         <mesh
-          filename="package://inspire_hand_description/meshes/visual/Link11.STL" />
-      </geometry>
-      <material
-        name="">
-        <color
-          rgba="1 1 1 1" />
-      </material>
-    </visual>
-    <collision>
-      <origin
-        xyz="0 0 0"
-        rpy="0 0 0" />
-      <geometry>
-        <mesh
-          filename="package://inspire_hand_description/meshes/visual/Link11.STL" />
+          filename="${pkg_address}/meshes/visual/Link11.STL" />
+      </geometry>
+      <material
+        name="">
+        <color
+          rgba="1 1 1 1" />
+      </material>
+    </visual>
+    <collision>
+      <origin
+        xyz="0 0 0"
+        rpy="0 0 0" />
+      <geometry>
+        <mesh
+          filename="${pkg_address}/meshes/visual/Link11.STL" />
       </geometry>
     </collision>
@@ -135,19 +135,19 @@
       <geometry>
         <mesh
-          filename="package://inspire_hand_description/meshes/visual/Link12.STL" />
-      </geometry>
-      <material
-        name="">
-        <color
-          rgba="1 1 1 1" />
-      </material>
-    </visual>
-    <collision>
-      <origin
-        xyz="0 0 0"
-        rpy="0 0 0" />
-      <geometry>
-        <mesh
-          filename="package://inspire_hand_description/meshes/visual/Link12.STL" />
+          filename="${pkg_address}/meshes/visual/Link12.STL" />
+      </geometry>
+      <material
+        name="">
+        <color
+          rgba="1 1 1 1" />
+      </material>
+    </visual>
+    <collision>
+      <origin
+        xyz="0 0 0"
+        rpy="0 0 0" />
+      <geometry>
+        <mesh
+          filename="${pkg_address}/meshes/visual/Link12.STL" />
       </geometry>
     </collision>
@@ -193,19 +193,19 @@
       <geometry>
         <mesh
-          filename="package://inspire_hand_description/meshes/visual/Link13.STL" />
-      </geometry>
-      <material
-        name="">
-        <color
-          rgba="1 1 1 1" />
-      </material>
-    </visual>
-    <collision>
-      <origin
-        xyz="0 0 0"
-        rpy="0 0 0" />
-      <geometry>
-        <mesh
-          filename="package://inspire_hand_description/meshes/visual/Link13.STL" />
+          filename="${pkg_address}/meshes/visual/Link13.STL" />
+      </geometry>
+      <material
+        name="">
+        <color
+          rgba="1 1 1 1" />
+      </material>
+    </visual>
+    <collision>
+      <origin
+        xyz="0 0 0"
+        rpy="0 0 0" />
+      <geometry>
+        <mesh
+          filename="${pkg_address}/meshes/visual/Link13.STL" />
       </geometry>
     </collision>
@@ -255,19 +255,19 @@
       <geometry>
         <mesh
-          filename="package://inspire_hand_description/meshes/visual/Link14.STL" />
-      </geometry>
-      <material
-        name="">
-        <color
-          rgba="1 1 1 1" />
-      </material>
-    </visual>
-    <collision>
-      <origin
-        xyz="0 0 0"
-        rpy="0 0 0" />
-      <geometry>
-        <mesh
-          filename="package://inspire_hand_description/meshes/visual/Link14.STL" />
+          filename="${pkg_address}/meshes/visual/Link14.STL" />
+      </geometry>
+      <material
+        name="">
+        <color
+          rgba="1 1 1 1" />
+      </material>
+    </visual>
+    <collision>
+      <origin
+        xyz="0 0 0"
+        rpy="0 0 0" />
+      <geometry>
+        <mesh
+          filename="${pkg_address}/meshes/visual/Link14.STL" />
       </geometry>
     </collision>
@@ -317,19 +317,19 @@
       <geometry>
         <mesh
-          filename="package://inspire_hand_description/meshes/visual/Link15.STL" />
-      </geometry>
-      <material
-        name="">
-        <color
-          rgba="1 1 1 1" />
-      </material>
-    </visual>
-    <collision>
-      <origin
-        xyz="0 0 0"
-        rpy="0 0 0" />
-      <geometry>
-        <mesh
-          filename="package://inspire_hand_description/meshes/visual/Link15.STL" />
+          filename="${pkg_address}/meshes/visual/Link15.STL" />
+      </geometry>
+      <material
+        name="">
+        <color
+          rgba="1 1 1 1" />
+      </material>
+    </visual>
+    <collision>
+      <origin
+        xyz="0 0 0"
+        rpy="0 0 0" />
+      <geometry>
+        <mesh
+          filename="${pkg_address}/meshes/visual/Link15.STL" />
       </geometry>
     </collision>
@@ -375,19 +375,19 @@
       <geometry>
         <mesh
-          filename="package://inspire_hand_description/meshes/visual/Link16.STL" />
-      </geometry>
-      <material
-        name="">
-        <color
-          rgba="1 1 1 1" />
-      </material>
-    </visual>
-    <collision>
-      <origin
-        xyz="0 0 0"
-        rpy="0 0 0" />
-      <geometry>
-        <mesh
-          filename="package://inspire_hand_description/meshes/visual/Link16.STL" />
+          filename="${pkg_address}/meshes/visual/Link16.STL" />
+      </geometry>
+      <material
+        name="">
+        <color
+          rgba="1 1 1 1" />
+      </material>
+    </visual>
+    <collision>
+      <origin
+        xyz="0 0 0"
+        rpy="0 0 0" />
+      <geometry>
+        <mesh
+          filename="${pkg_address}/meshes/visual/Link16.STL" />
       </geometry>
     </collision>
@@ -437,19 +437,19 @@
       <geometry>
         <mesh
-          filename="package://inspire_hand_description/meshes/visual/Link17.STL" />
-      </geometry>
-      <material
-        name="">
-        <color
-          rgba="1 1 1 1" />
-      </material>
-    </visual>
-    <collision>
-      <origin
-        xyz="0 0 0"
-        rpy="0 0 0" />
-      <geometry>
-        <mesh
-          filename="package://inspire_hand_description/meshes/visual/Link17.STL" />
+          filename="${pkg_address}/meshes/visual/Link17.STL" />
+      </geometry>
+      <material
+        name="">
+        <color
+          rgba="1 1 1 1" />
+      </material>
+    </visual>
+    <collision>
+      <origin
+        xyz="0 0 0"
+        rpy="0 0 0" />
+      <geometry>
+        <mesh
+          filename="${pkg_address}/meshes/visual/Link17.STL" />
       </geometry>
     </collision>
@@ -495,19 +495,19 @@
       <geometry>
         <mesh
-          filename="package://inspire_hand_description/meshes/visual/Link18.STL" />
-      </geometry>
-      <material
-        name="">
-        <color
-          rgba="1 1 1 1" />
-      </material>
-    </visual>
-    <collision>
-      <origin
-        xyz="0 0 0"
-        rpy="0 0 0" />
-      <geometry>
-        <mesh
-          filename="package://inspire_hand_description/meshes/visual/Link18.STL" />
+          filename="${pkg_address}/meshes/visual/Link18.STL" />
+      </geometry>
+      <material
+        name="">
+        <color
+          rgba="1 1 1 1" />
+      </material>
+    </visual>
+    <collision>
+      <origin
+        xyz="0 0 0"
+        rpy="0 0 0" />
+      <geometry>
+        <mesh
+          filename="${pkg_address}/meshes/visual/Link18.STL" />
       </geometry>
     </collision>
@@ -557,19 +557,19 @@
       <geometry>
         <mesh
-          filename="package://inspire_hand_description/meshes/visual/Link19.STL" />
-      </geometry>
-      <material
-        name="">
-        <color
-          rgba="1 1 1 1" />
-      </material>
-    </visual>
-    <collision>
-      <origin
-        xyz="0 0 0"
-        rpy="0 0 0" />
-      <geometry>
-        <mesh
-          filename="package://inspire_hand_description/meshes/visual/Link19.STL" />
+          filename="${pkg_address}/meshes/visual/Link19.STL" />
+      </geometry>
+      <material
+        name="">
+        <color
+          rgba="1 1 1 1" />
+      </material>
+    </visual>
+    <collision>
+      <origin
+        xyz="0 0 0"
+        rpy="0 0 0" />
+      <geometry>
+        <mesh
+          filename="${pkg_address}/meshes/visual/Link19.STL" />
       </geometry>
     </collision>
@@ -615,19 +615,19 @@
       <geometry>
         <mesh
-          filename="package://inspire_hand_description/meshes/visual/Link20.STL" />
-      </geometry>
-      <material
-        name="">
-        <color
-          rgba="1 1 1 1" />
-      </material>
-    </visual>
-    <collision>
-      <origin
-        xyz="0 0 0"
-        rpy="0 0 0" />
-      <geometry>
-        <mesh
-          filename="package://inspire_hand_description/meshes/visual/Link20.STL" />
+          filename="${pkg_address}/meshes/visual/Link20.STL" />
+      </geometry>
+      <material
+        name="">
+        <color
+          rgba="1 1 1 1" />
+      </material>
+    </visual>
+    <collision>
+      <origin
+        xyz="0 0 0"
+        rpy="0 0 0" />
+      <geometry>
+        <mesh
+          filename="${pkg_address}/meshes/visual/Link20.STL" />
       </geometry>
     </collision>
@@ -677,19 +677,19 @@
       <geometry>
         <mesh
-          filename="package://inspire_hand_description/meshes/visual/Link21.STL" />
-      </geometry>
-      <material
-        name="">
-        <color
-          rgba="1 1 1 1" />
-      </material>
-    </visual>
-    <collision>
-      <origin
-        xyz="0 0 0"
-        rpy="0 0 0" />
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
File: robot_description/robotiq_gripper_description/urdf/gazebo/robotiq_gripper_gazebo.urdf.xacro (robot description, xacro)
@@ -24,5 +24,5 @@
       <origin rpy="0 0 0" xyz="0 0 0"/>
       <geometry>
-        <mesh filename="package://robotiq_gripper_description/meshes/visual/hand-e.dae" scale="1.0 1.0 1.0"/>
+        <mesh filename="${pkg_address}/meshes/visual/hand-e.dae" scale="1.0 1.0 1.0"/>
       </geometry>
       <material name="Dark">
@@ -33,5 +33,5 @@
       <origin rpy="0 0 0" xyz="0 0 0"/>
       <geometry>
-        <mesh filename="package://robotiq_gripper_description/meshes/visual/hand-e.dae" scale="1.0 1.0 1.0"/>
+        <mesh filename="${pkg_address}/meshes/visual/hand-e.dae" scale="1.0 1.0 1.0"/>
       </geometry>
     </collision>
@@ -46,5 +46,5 @@
       <origin rpy="0 0 0" xyz="0 0 0"/>
       <geometry>
-        <mesh filename="package://robotiq_gripper_description/meshes/visual/finger_1.dae" scale="1.0 1.0 1.0"/>
+        <mesh filename="${pkg_address}/meshes/visual/finger_1.dae" scale="1.0 1.0 1.0"/>
       </geometry>
       <material name="DarkGray">
@@ -55,5 +55,5 @@
       <origin rpy="0 0 0" xyz="0 0 0"/>
       <geometry>
-        <mesh filename="package://robotiq_gripper_description/meshes/visual/finger_1.dae" scale="1.0 1.0 1.0"/>
+        <mesh filename="${pkg_address}/meshes/visual/finger_1.dae" scale="1.0 1.0 1.0"/>
       </geometry>
     </collision>
@@ -68,5 +68,5 @@
       <origin rpy="0 0 0" xyz="0 0 0"/>
       <geometry>
-        <mesh filename="package://robotiq_gripper_description/meshes/visual/finger_2.dae" scale="1.0 1.0 1.0"/>
+        <mesh filename="${pkg_address}/meshes/visual/finger_2.dae" scale="1.0 1.0 1.0"/>
       </geometry>
       <material name="DarkGray">
@@ -77,5 +77,5 @@
       <origin rpy="0 0 0" xyz="0 0 0"/>
       <geometry>
-        <mesh filename="package://robotiq_gripper_description/meshes/visual/finger_2.dae" scale="1.0 1.0 1.0"/>
+        <mesh filename="${pkg_address}/meshes/visual/finger_2.dae" scale="1.0 1.0 1.0"/>
       </geometry>
     </collision>

File: robot_description/t1_description/urdf/gazebo/t1_gazebo.urdf.xacro (robot description, xacro)
@@ -40,5 +40,5 @@
       <geometry>
         <mesh
-          filename="package://t1_description/meshes/base_link.STL" />
+          filename="${pkg_address}/meshes/base_link.STL" />
       </geometry>
       <material
@@ -54,5 +54,5 @@
       <geometry>
         <mesh
-          filename="package://t1_description/meshes/base_link.STL" />
+          filename="${pkg_address}/meshes/base_link.STL" />
       </geometry>
     </collision>
@@ -80,5 +80,5 @@
       <geometry>
         <mesh
-          filename="package://t1_description/meshes/Link-Body.STL" />
+          filename="${pkg_address}/meshes/Link-Body.STL" />
       </geometry>
       <material
@@ -94,5 +94,5 @@
       <geometry>
         <mesh
-          filename="package://t1_description/meshes/Link-Body.STL" />
+          filename="${pkg_address}/meshes/Link-Body.STL" />
       </geometry>
     </collision>
@@ -138,5 +138,5 @@
       <geometry>
         <mesh
-          filename="package://t1_description/meshes/link-R0.STL" />
+          filename="${pkg_address}/meshes/link-R0.STL" />
       </geometry>
       <material
@@ -152,5 +152,5 @@
       <geometry>
         <mesh
-          filename="package://t1_description/meshes/link-R0.STL" />
+          filename="${pkg_address}/meshes/link-R0.STL" />
       </geometry>
     </collision>
@@ -191,5 +191,5 @@
       <geometry>
         <mesh
-          filename="package://t1_description/meshes/link-R1.STL" />
+          filename="${pkg_address}/meshes/link-R1.STL" />
       </geometry>
       <material
@@ -205,5 +205,5 @@
       <geometry>
         <mesh
-          filename="package://t1_description/meshes/link-R1.STL" />
+          filename="${pkg_address}/meshes/link-R1.STL" />
       </geometry>
     </collision>
@@ -249,5 +249,5 @@
       <geometry>
         <mesh
-          filename="package://t1_description/meshes/link-R2.STL" />
+          filename="${pkg_address}/meshes/link-R2.STL" />
       </geometry>
       <material
@@ -263,5 +263,5 @@
       <geometry>
         <mesh
-          filename="package://t1_description/meshes/link-R2.STL" />
+          filename="${pkg_address}/meshes/link-R2.STL" />
       </geometry>
     </collision>
@@ -307,5 +307,5 @@
       <geometry>
         <mesh
-          filename="package://t1_description/meshes/link-R3.STL" />
+          filename="${pkg_address}/meshes/link-R3.STL" />
       </geometry>
       <material
@@ -321,5 +321,5 @@
       <geometry>
         <mesh
-          filename="package://t1_description/meshes/link-R3.STL" />
+          filename="${pkg_address}/meshes/link-R3.STL" />
       </geometry>
     </collision>
@@ -365,5 +365,5 @@
       <geometry>
         <mesh
-          filename="package://t1_description/meshes/link-R4.STL" />
+          filename="${pkg_address}/meshes/link-R4.STL" />
       </geometry>
       <material
@@ -379,5 +379,5 @@
       <geometry>
         <mesh
-          filename="package://t1_description/meshes/link-R4.STL" />
+          filename="${pkg_address}/meshes/link-R4.STL" />
       </geometry>
     </collision>
@@ -423,5 +423,5 @@
       <geometry>
         <mesh
-          filename="package://t1_description/meshes/link-R5.STL" />
+          filename="${pkg_address}/meshes/link-R5.STL" />
       </geometry>
       <material
@@ -437,5 +437,5 @@
       <geometry>
         <mesh
-          filename="package://t1_description/meshes/link-R5.STL" />
+          filename="${pkg_address}/meshes/link-R5.STL" />
       </geometry>
     </collision>
@@ -481,5 +481,5 @@
       <geometry>
         <mesh
-          filename="package://t1_description/meshes/link-R6.STL" />
+          filename="${pkg_address}/meshes/link-R6.STL" />
       </geometry>
       <material
@@ -495,5 +495,5 @@
       <geometry>
         <mesh
-          filename="package://t1_description/meshes/link-R6.STL" />
+          filename="${pkg_address}/meshes/link-R6.STL" />
       </geometry>
     </collision>
@@ -539,5 +539,5 @@
       <geometry>
         <mesh
-          filename="package://t1_description/meshes/link-R7.STL" />
+          filename="${pkg_address}/meshes/link-R7.STL" />
       </geometry>
       <material
@@ -553,5 +553,5 @@
       <geometry>
         <mesh
-          filename="package://t1_description/meshes/link-R7.STL" />
+          filename="${pkg_address}/meshes/link-R7.STL" />
       </geometry>
     </collision>
@@ -597,5 +597,5 @@
       <geometry>
         <mesh
-          filename="package://t1_description/meshes/link-Rtool.STL" />
+          filename="${pkg_address}/meshes/link-Rtool.STL" />
       </geometry>
       <material
@@ -611,5 +611,5 @@
       <geometry>
         <mesh
-          filename="package://t1_description/meshes/link-Rtool.STL" />
+          filename="${pkg_address}/meshes/link-Rtool.STL" />
       </geometry>
     </collision>
@@ -650,5 +650,5 @@
       <geometry>
         <mesh
-          filename="package://t1_description/meshes/link-L0.STL" />
+          filename="${pkg_address}/meshes/link-L0.STL" />
       </geometry>
       <material
@@ -664,5 +664,5 @@
       <geometry>
         <mesh
-          filename="package://t1_description/meshes/link-L0.STL" />
+          filename="${pkg_address}/meshes/link-L0.STL" />
       </geometry>
     </collision>
@@ -703,5 +703,5 @@
       <geometry>
         <mesh
-          filename="package://t1_description/meshes/link-L1.STL" />
+          filename="${pkg_address}/meshes/link-L1.STL" />
       </geometry>
       <material
@@ -717,5 +717,5 @@
       <geometry>
         <mesh
-          filename="package://t1_description/meshes/link-L1.STL" />
+          filename="${pkg_address}/meshes/link-L1.STL" />
       </geometry>
     </collision>
@@ -761,5 +761,5 @@
       <geometry>
         <mesh
-          filename="package://t1_description/meshes/link-L2.STL" />
+          filename="${pkg_address}/meshes/link-L2.STL" />
       </geometry>
       <material
@@ -775,5 +775,5 @@
       <geometry>
         <mesh
-          filename="package://t1_description/meshes/link-L2.STL" />
+          filename="${pkg_address}/meshes/link-L2.STL" />
       </geometry>
     </collision>
@@ -819,5 +819,5 @@
       <geometry>
         <mesh
-          filename="package://t1_description/meshes/link-L3.STL" />
+          filename="${pkg_address}/meshes/link-L3.STL" />
       </geometry>
       <material
@@ -833,5 +833,5 @@
       <geometry>
         <mesh
-          filename="package://t1_description/meshes/link-L3.STL" />
+          filename="${pkg_address}/meshes/link-L3.STL" />
       </geometry>
     </collision>
@@ -877,5 +877,5 @@
       <geometry>
         <mesh
-          filename="package://t1_description/meshes/link-L4.STL" />
+          filename="${pkg_address}/meshes/link-L4.STL" />
       </geometry>
       <material
@@ -891,5 +891,5 @@
       <geometry>
         <mesh
-          filename="package://t1_description/meshes/link-L4.STL" />
+          filename="${pkg_address}/meshes/link-L4.STL" />
       </geometry>
     </collision>
@@ -935,5 +935,5 @@
       <geometry>
         <mesh
-          filename="package://t1_description/meshes/link-L5.STL" />
+          filename="${pkg_address}/meshes/link-L5.STL" />
       </geometry>
       <material
@@ -949,5 +949,5 @@
       <geometry>
         <mesh
-          filename="package://t1_description/meshes/link-L5.STL" />
+          filename="${pkg_address}/meshes/link-L5.STL" />
       </geometry>
     </collision>
@@ -993,5 +993,5 @@
       <geometry>
         <mesh
-          filename="package://t1_description/meshes/link-L6.STL" />
+          filename="${pkg_address}/meshes/link-L6.STL" />
       </geometry>
       <material
@@ -1007,5 +1007,5 @@
       <geometry>
         <mesh
-          filename="package://t1_description/meshes/link-L6.STL" />
+          filename="${pkg_address}/meshes/link-L6.STL" />
       </geometry>
     </collision>
@@ -1051,5 +1051,5 @@
       <geometry>
         <mesh
-          filename="package://t1_description/meshes/link-L7.STL" />
+          filename="${pkg_address}/meshes/link-L7.STL" />
       </geometry>
       <material
@@ -1065,5 +1065,5 @@
       <geometry>
         <mesh
-          filename="package://t1_description/meshes/link-L7.STL" />
+          filename="${pkg_address}/meshes/link-L7.STL" />
       </geometry>
     </collision>
@@ -1109,5 +1109,5 @@
       <geometry>
         <mesh
-          filename="package://t1_description/meshes/link-Ltool.STL" />
+          filename="${pkg_address}/meshes/link-Ltool.STL" />
       </geometry>
       <material
@@ -1123,5 +1123,5 @@
       <geometry>
         <mesh
-          filename="package://t1_description/meshes/link-Ltool.STL" />
+          filename="${pkg_address}/meshes/link-Ltool.STL" />
       </geometry>
     </collision>
@@ -1162,5 +1162,5 @@
       <geometry>
         <mesh
-          filename="package://t1_description/meshes/link-H1.STL" />
+          filename="${pkg_address}/meshes/link-H1.STL" />
       </geometry>
       <material
@@ -1176,5 +1176,5 @@
       <geometry>
         <mesh
-          filename="package://t1_description/meshes/link-H1.STL" />
+          filename="${pkg_address}/meshes/link-H1.STL" />
       </geometry>
     </collision>
@@ -1220,5 +1220,5 @@
       <geometry>
         <mesh
-          filename="package://t1_description/meshes/link-H2.STL" />
+          filename="${pkg_address}/meshes/link-H2.STL" />
       </geometry>
       <material
@@ -1234,5 +1234,5 @@
       <geometry>
         <mesh
-          filename="package://t1_description/meshes/link-H2.STL" />
+          filename="${pkg_address}/meshes/link-H2.STL" />
       </geometry>
     </collision>
@@ -1278,5 +1278,5 @@
       <geometry>
         <mesh
-          filename="package://t1_description/meshes/link-realsense.STL" />
+          filename="${pkg_address}/meshes/link-realsense.STL" />
       </geometry>
       <material
@@ -1292,5 +1292,5 @@
       <geometry>
         <mesh
-          filename="package://t1_description/meshes/link-realsense.STL" />
+          filename="${pkg_address}/meshes/link-realsense.STL" />
       </geometry>
     </collision>
@@ -1331,5 +1331,5 @@
       <geometry>
         <mesh
-          filename="package://t1_description/meshes/link-zed.STL" />
+          filename="${pkg_address}/meshes/link-zed.STL" />
       </geometry>
       <material
@@ -1345,5 +1345,5 @@
       <geometry>
         <mesh
-          filename="package://t1_description/meshes/link-zed.STL" />
+          filename="${pkg_address}/meshes/link-zed.STL" />
       </geometry>
     </collision>
