Commit message: finish moveXYZW_action, modify t1_description/t1_movit_driver/gazebo_driver, repair t1_tf, moveit.rviz

File: robot_description/t1_description/urdf/external_devices_config.xacro (robot description, xacro)
@@ -1,21 +1,15 @@
 <?xml version="1.0" encoding="utf-8"?>
 <robot name = "external_devices" xmlns:xacro="http://ros.org/wiki/xacro">
-  <xacro:macro name="external_device_config" params="if_add_external_device">
-    <xacro:if value="${if_add_external_device}">
-      <xacro:include filename="$(find inspire_hand_description)/urdf/inspire_hand.urdf.xacro"/>
-      <xacro:include filename="$(find robotiq_gripper_description)/urdf/robotiq_gripper.urdf.xacro"/>
-      <joint name="gripper_connect_joint" type="fixed">
-        <origin xyz="0 0 0" rpy="0 0 1.57" />
-        <!-- <origin xyz="0 0 0.00695" rpy="0 0 0" /> -->
-        <parent link="link-Ltool"/>
-        <child link="hand_e_link"/>
-      </joint>
-      <joint name="hand_connect_joint" type="fixed">
-        <!-- <origin xyz="0 0 0" rpy="-1.57 0 -1.57" /> -->
-        <origin xyz="0 0 0" rpy="-1.57 0 0" />
-        <parent link="link-Rtool"/>
-        <child link="R_hand_base_link"/>
-      </joint>
-    </xacro:if>
-  </xacro:macro>
+  <joint name="gripper_connect_joint" type="fixed">
+    <origin xyz="0 0 0" rpy="0 0 1.57" />
+    <!-- <origin xyz="0 0 0.00695" rpy="0 0 0" /> -->
+    <parent link="link-Ltool"/>
+    <child link="hand_e_link"/>
+  </joint>
+  <joint name="hand_connect_joint" type="fixed">
+    <!-- <origin xyz="0 0 0" rpy="-1.57 0 -1.57" /> -->
+    <origin xyz="0 0 0" rpy="-1.57 0 0" />
+    <parent link="link-Rtool"/>
+    <child link="R_hand_base_link"/>
+  </joint>
 </robot>

File: robot_description/t1_description/urdf/gazebo_config.xacro (robot description, xacro)
@@ -1,12 +1,8 @@
 <?xml version="1.0" encoding="utf-8"?>
 <robot name = "h1" xmlns:xacro="http://ros.org/wiki/xacro">
-  <xacro:macro name="gazebo_config" params="sim_gazebo_classic">
-    <xacro:if value="${sim_gazebo_classic}">
-      <link name="world"/>
-      <joint name="fixed" type="fixed">
-        <parent link="world"/>
-        <child link="fake_link"/>
-      </joint>
-    </xacro:if>
-  </xacro:macro>
+    <link name="world"/>
+    <joint name="fixed" type="fixed">
+      <parent link="world"/>
+      <child link="fake_link"/>
+    </joint>
 </robot>

File: robot_description/t1_description/urdf/t1.xacro (robot description, xacro)
@@ -8,9 +8,17 @@
   <xacro:arg name="if_add_external_device" default="false" />
   <xacro:arg name="external_device_dof" default="7" />
-  <xacro:include filename="$(find t1_description)/urdf/t1.urdf.xacro"/>
-  <xacro:include filename="$(find t1_description)/urdf/gazebo_config.xacro"/>
-  <xacro:include filename="$(find t1_description)/urdf/external_devices_config.xacro"/>
-  <xacro:external_device_config if_add_external_device="$(arg if_add_external_device)"/>
-  <xacro:gazebo_config sim_gazebo_classic="$(arg sim_gazebo_classic)"/>
+  <xacro:if value="$(arg sim_gazebo_classic)">
+    <xacro:include filename="$(find t1_description)/urdf/gazebo/t1_gazebo.urdf.xacro"/>
+    <xacro:include filename="$(find inspire_hand_description)/urdf/gazebo/inspire_hand_gazebo.urdf.xacro"/>
+    <xacro:include filename="$(find robotiq_gripper_description)/urdf/gazebo/robotiq_gripper_gazebo.urdf.xacro"/>
+    <xacro:include filename="$(find t1_description)/urdf/external_devices_config.xacro"/>
+    <xacro:include filename="$(find t1_description)/urdf/gazebo_config.xacro"/>
+  </xacro:if>
+  <xacro:unless value="$(arg sim_gazebo_classic)">
+    <xacro:include filename="$(find t1_description)/urdf/t1.urdf.xacro"/>
+    <xacro:include filename="$(find inspire_hand_description)/urdf/inspire_hand.urdf.xacro"/>
+    <xacro:include filename="$(find robotiq_gripper_description)/urdf/robotiq_gripper.urdf.xacro"/>
+    <xacro:include filename="$(find t1_description)/urdf/external_devices_config.xacro"/>
+  </xacro:unless>
   <xacro:include filename="$(find t1_description)/urdf/t1_robot_ros2_control.xacro"/>
   <xacro:t1_robot_ros2_control_config

File: robot_description/t1_description/urdf/t1_robot.urdf.xacro (robot description, xacro)
@@ -1,7 +1,7 @@
 <?xml version="1.0" encoding="UTF-8"?>
 <robot name="t1_robot" xmlns:xacro="http://wiki.ros.org/xacro" >
-    <xacro:arg name="if_add_external_device" default="true" />
     <xacro:include filename="$(find t1_description)/urdf/t1.urdf.xacro"/>
+    <xacro:include filename="$(find inspire_hand_description)/urdf/inspire_hand.urdf.xacro"/>
+    <xacro:include filename="$(find robotiq_gripper_description)/urdf/robotiq_gripper.urdf.xacro"/>
     <xacro:include filename="$(find t1_description)/urdf/external_devices_config.xacro"/>
-    <xacro:external_device_config if_add_external_device="$(arg if_add_external_device)"/>
 </robot>

File: robot_description/t1_description/urdf/t1_robot_ros2_control.xacro (robot description, xacro)
@@ -8,5 +8,5 @@
         </plugin>
       </gazebo>
-      <!-- <xacro:macro name ="link_reference" params="link_name material_">
+      <xacro:macro name ="link_reference" params="link_name material_">
         <gazebo reference="${link_name}">
           <material>${material_}</material>
@@ -14,6 +14,5 @@
       </xacro:macro>
       <xacro:link_reference link_name="base_link" material_= "Gazebo/DarkGrey"/>
-      <xacro:link_reference link_name="link-J1" material_= "Gazebo/Orange"/>
-      <xacro:link_reference link_name="link-Body" material_= "Gazebo/DarkGrey"/>
+      <xacro:link_reference link_name="link-Body" material_= "Gazebo/Orange"/>
       <xacro:link_reference link_name="link-L0" material_= "Gazebo/White"/>
       <xacro:link_reference link_name="link-L1" material_= "Gazebo/Grey"/>
@@ -33,5 +32,5 @@
       <xacro:link_reference link_name="link-R7" material_= "Gazebo/Grey"/>
       <xacro:link_reference link_name="link-H0" material_= "Gazebo/White"/>
-      <xacro:link_reference link_name="link-H1" material_= "Gazebo/Grey"/> -->
+      <xacro:link_reference link_name="link-H1" material_= "Gazebo/Grey"/>
     </xacro:if>
     <ros2_control name="h1_robot_ros2_control" type="system">

File: robot_moveit_config/t1_robot_moveit_config/config/t1_robot.urdf.xacro (robot description, xacro)
@@ -1,13 +1,7 @@
 <?xml version="1.0"?>
 <robot xmlns:xacro="http://www.ros.org/wiki/xacro" name="t1_robot">
-    <xacro:arg name="initial_positions_file" default="initial_positions.yaml" />
-    <xacro:arg name="sim_gazebo_classic" default="true" />
-    <!-- Import t1_robot urdf file -->
-    <xacro:include filename="$(find t1_description)/urdf/t1_robot.urdf.xacro" />
-    <!-- Import control_xacro -->
-    <xacro:include filename="t1_robot.ros2_control.xacro" />
-    <!-- Import control_xacro -->
-    <xacro:include filename="$(find t1_description)/urdf/gazebo_config.xacro"/>
-    <xacro:gazebo_config sim_gazebo_classic="$(arg sim_gazebo_classic)"/>
-    <xacro:t1_robot_ros2_control name="FakeSystem" initial_positions_file="$(arg initial_positions_file)"/>
+    <!-- <xacro:arg name="initial_positions_file" default="initial_positions.yaml" /> -->
+    <!-- <xacro:include filename="$(find t1_description)/urdf/t1_robot.urdf.xacro" />
+    <xacro:include filename="t1_robot.ros2_control.xacro" /> -->
+    <!-- <xacro:t1_robot_ros2_control name="FakeSystem" initial_positions_file="$(arg initial_positions_file)"/> -->
 </robot>
